File: VFDFFT.kicad_sch (KiCad schematic)
At the start: 185 parts, among them J1 USB_C_Receptacle_USB2.0, J2 BATT, J3 FILAMENT+, J4 VFD_SIG, Q1 IRL7486MTRPBF, Q2 ASDM30DN40E, Q3 ASDM30DN40E, Q4 HSCB2903, Q5 HSCB2903, Q6 AP6800, Q7 FS5N10S, Q8 FS5N10S, U1 IP2368, U10 TPS61170, U11 TPS61170, U2 78L05_SOT23, U3 TPS40305, U4 LM3478, U5 LM3478, U6 STM32F205VBTx, U7 AP6181, U8 HDC1080, U9 OPT3001DNPR, X1 SX1M32.768KM10F30TNN, Y1 26M, Y2 24M

Commit message: assign footprint 30%
Parts:
- AE1: footprint (none) -> Resistor_SMD:R_1206_3216Metric
- C1: footprint (none) -> Resistor_SMD:R_0603_1608Metric
- C10, C11, C12, C13, C18, C19, C20, C21, C22, C23, C24, C25, C26, C27, C28, C29, C32, C33, C34, C35, C37, C38, C40, C41, C43, C44, C45, C46, C47, C48, C49, C50, C51, C52, C53, C54, C55, C56, C57, C58, C59, C60, C61, C62, C63, C64, C65, C66, C7, C8, C9: footprint (none) -> Capacitor_SMD:C_0603_1608Metric
- C14, C2: footprint (none) -> Capacitor_Tantalum_SMD:CP_EIA-7343-30_AVX-N
- C15, C16, C17, C3, C30, C4, C5, C6: footprint (none) -> Capacitor_SMD:C_0805_2012Metric
- C31, C39: footprint (none) -> Capacitor_Tantalum_SMD:CP_EIA-6032-28_Kemet-C
- C36, C42: footprint (none) -> Capacitor_SMD:CP_Elec_6.3x5.9

Commit message: complete almost schem
Parts:
- removed U6: STM32F205VBTx, Package_QFP:LQFP-100_14x14mm_P0.5mm, symbol MCU_ST_STM32F2:STM32F205VBTx
- added C76: 100nF, symbol Device:C_Small
- added C77: 10uF, symbol Device:C_Small
- added C78: 22uF, symbol Device:C_Small
- added J5: USB_A, symbol Connector:USB_A
- added L9: 2.2uH, symbol Device:L_Small
- added R58: 10K, symbol Device:R_Small
- added R59: 953K, symbol Device:R_Small
- added R60: 180K, symbol Device:R_Small
- added R61: 100K, symbol Device:R_Small
- added U12: W25Q128JVS, Package_SO:SOIC-8_5.23x5.23mm_P1.27mm, symbol Memory_Flash:W25Q128JVS
- added U13: TPS62170DSG, Package_SON:WSON-8-1EP_2x2mm_P0.5mm_EP0.9x1.6mm_ThermalVias, symbol Regulator_Switching:TPS62170DSG
- added U6: STM32F446VETx, Package_QFP:LQFP-100_14x14mm_P0.5mm, symbol MCU_ST_STM32F4:STM32F446VETx
Connections:
- net +3V3: now also C76.2, R58.1, U12.8 (VCC), U6.100 (VDD), U6.11 (VDD), U6.19 (VDD), U6.21 (VREF+), U6.22 (VDDA), U6.28 (VDD), U6.50 (VDD), U6.6 (VBAT), U6.75 (VDD)
- net +BATT: now also C77.1, U13.2 (VIN), U13.3 (EN)
- net DAC1: now also U6.29 (PA4)
- net DAC2: now also U6.30 (PA5)
- net GND: now also C76.1, C77.2, C78.2, J5.4 (GND), J5.5 (Shield), R60.2, U12.4 (GND), U13.1 (PGND), U13.4 (AGND), U13.9 (PAD), U6.10 (VSS), U6.20 (VSSA), U6.27 (VSS), U6.49 (VSS), U6.74 (VSS), U6.99 (VSS)
- net HUM_SCK: now also U6.67 (PA8)
- net HUM_SDA: now also U6.66 (PC9)
- net MIC_SCK: now also U6.89 (PB3)
- net MIC_SD: now also U6.32 (PA7)
- net MIC_WS: now also U6.77 (PA15)
- net OPT_SCL: now also U6.47 (PB10)
- net OPT_SDA: now also U6.80 (PC12)
- net SWCLK: now also U6.76 (PA14)
- net SWDIO: now also U6.72 (PA13)
- net VFD_CLK: now also U6.52 (PB13)
- net VFD_CS: now also U6.15 (PC0)
- net VFD_DATA: now also U6.16 (PC1)
- net VFD_RST: now also U6.51 (PB12)
- net WL_CLK: now also U6.37 (PB2)
- net WL_CMD: now also U6.83 (PD2)
- net WL_D0: now also U6.65 (PC8)
- net WL_D1: now also U6.35 (PB0)
- net WL_D2: now also U6.36 (PB1)
- net WL_D3: now also U6.79 (PC11)
- net at C64.2, R46.1: now also U6.14 (NRST)
- net at C66.2, Y2.1: now also U6.13 (PH1)
- net at C65.2, Y2.2: now also U6.12 (PH0)
- net at C60.2: now also U6.48 (VCAP_1)
- net at C61.2: now also U6.73 (VCAP_2)
- net at R45.2: now also U6.94 (BOOT0)
- new net: R59.2, R60.1, U13.5 (FB)
- new net: J5.2 (D-), U6.53 (PB14)
- new net: J5.3 (D+), U6.54 (PB15)
- new net: R61.2, U13.8 (PG)
- new net: L9.1, U13.7 (SW)
- new net +5V: C78.1, J5.1 (VBUS), L9.2, R59.1, R61.1, U13.6 (VOS)
- new net FLASH_CS: R58.2, U12.1 (~{CS})
- new net FLASH_IO0: U12.5 (DI(IO0)), U6.58 (PD11)
- new net FLASH_IO1: U12.2 (DO(IO1)), U6.59 (PD12)
- new net FLASH_IO2: U12.3 (IO2), U6.1 (PE2)
- new net FLASH_IO3: U12.7 (IO3), U6.24 (PA1)
- new net FLASH_SCK: U12.6 (CLK), U6.84 (PD3), U6.92 (PB6)
- no-connect marks 24 -> 23
Other:
- moved on the sheet: C60, C61

Commit message: file sync
Parts:
- added C79, C80, C81, C82: 100nF, symbol Device:C_Small
- added D13: ADR5040, symbol Device:D_Zener
- added J10, J8, J9: Conn_01x02_Pin, symbol Connector:Conn_01x02_Pin
- added J6, J7: Conn_01x03_Socket, symbol Connector:Conn_01x03_Socket
- added Q10, Q11, Q9: AO3400A, Package_TO_SOT_SMD:SOT-23, symbol Transistor_FET:AO3400A
- added R62, R63, R64, R65, R66, R67, R68, R71, R72, R76, R77, R79: 10K, symbol Device:R_Small
- added R69, R70, R73, R74: 20K, symbol Device:R_Small
- added R75, R78, R80: 1M, symbol Device:R_Small
- added U14: LM358, symbol Amplifier_Operational:LM358
- added U15: LM324, symbol Amplifier_Operational:LM324
Connections:
- net FLASH_CS: now also U6.92 (PB6)
- net FLASH_SCK: no longer U6.92 (PB6)
- net GND: now also C80.1, C82.1, U14.4 (V-), U15.11 (V-)
- net GNDA: now also C70.2, C71.1, D11.1 (K), R53.1, C79.2, C80.2, C81.2, C82.2, D13.2 (A), J6.2 (Pin_2), J7.2 (Pin_2), R69.2, R73.2, U14.5 (+), U15.3 (+); no longer C72.1, C73.2, D12.1 (K), R55.1
- net VDDA: now also C72.1, C73.2, D12.1 (K), R55.1, C79.1, C81.1, R62.1, U14.8 (V+), U15.4 (V+); no longer C70.2, C71.1, D11.1 (K), R53.1
- new net: R75.1, R76.1
- new net: R72.1, R73.1, U15.10 (+)
- new net: J8.2 (Pin_2), Q9.2 (S), R75.2
- new net: J9.2 (Pin_2), Q10.2 (S), R78.2
- new net: J9.1 (Pin_1), Q10.3 (D)
- new net: R65.1, R66.2, U15.2 (-)
- new net: J8.1 (Pin_1), Q9.3 (D)
- new net: R67.1, R69.1, U15.5 (+)
- new net: R71.1, R74.2, U15.9 (-)
- new net: R63.1, R64.2, U14.6 (-)
- new net: R79.1, R80.1
- new net: R77.1, R78.1
- new net: J10.1 (Pin_1), Q11.3 (D)
- new net: J10.2 (Pin_2), Q11.2 (S), R80.2
- new net: R68.1, R70.2, U15.6 (-)
- new net L: R71.2
- new net L+: J6.1 (Pin_1), R63.2, R74.1, U15.8
- new net L-: J6.3 (Pin_3), R64.1, U14.7
- new net LB: Q11.1 (G), R79.2
- new net LG: Q10.1 (G), R77.2
- new net LR: Q9.1 (G), R76.2
- new net R: R68.2
- new net R+: J7.1 (Pin_1), R65.2, R70.1, U15.7
- new net R-: J7.3 (Pin_3), R66.1, U15.1
- new net REF_B: R67.2, R72.2, U14.1, U14.2 (-)
- new net VS: D13.1 (K), R62.2, U14.3 (+)

Commit message: schem complete
Parts:
- added C83: 2.2nF, Capacitor_SMD:C_0603_1608Metric, symbol Device:C_Small
- added C84: 4pF, Capacitor_SMD:C_0603_1608Metric, symbol Device:C_Small
- added C85: 68uF, Capacitor_Tantalum_SMD:CP_EIA-6032-28_Kemet-C, symbol Device:C_Polarized_Small
- added C86: 10pF, Capacitor_SMD:C_0603_1608Metric, symbol Device:C_Small
- added C87, C90, C91: 100nF, Capacitor_SMD:C_0603_1608Metric, symbol Device:C_Small
- added C88: 22uF, Capacitor_SMD:CP_Elec_6.3x5.9, symbol Device:C_Polarized_Small
- added C89: 100uF, Capacitor_SMD:C_0805_2012Metric, symbol Device:C_Polarized_Small
- added D14: LBAT46T1G, symbol Device:D_Schottky_Small
- added D15, D16: 1V/200mA, symbol Device:D_Schottky_Small
- added D17: D_Zener_Small, symbol Device:D_Zener_Small
- added J11: Conn_01x02_Male, symbol Connector:Conn_01x02_Male
- added L10: BKW0805UCR12JST, symbol Device:L_Small
- added L11: CBC3225T220KR, symbol Device:L_Small
- added Q12: FS5N10S, symbol Device:Q_NMOS_GSD
- added R81: 20K, symbol Device:R_Small
- added R82: 12K1, symbol Device:R_Small
- added R83: 100, symbol Device:R_Small
- added R84: 75m, symbol Device:R_Small
- added R85: 11K, symbol Device:R_Small
- added R86, R88: 1K, symbol Device:R_Small
- added R87: 14K, symbol Device:R_Small
- added R89: 4K02, symbol Device:R_Small
- added U16: LM3478, symbol Project_Symbols:LM3478
- added U17: LM2738, symbol Project_Symbols:LM2738
- added U18: LTC1446, symbol Analog_DAC:LTC1446
Connections:
- net +5V: now also U18.7 (VCC)
- net +BATT: now also C85.1, C87.2, L10.1, U16.8 (VIN)
- net GND: now also C84.1, C85.2, C86.1, C87.1, C88.2, C89.2, C91.1, D15.2 (A), D17.2 (A), J11.2 (Pin_2), R81.1, R82.2, R84.2, R86.1, R88.1, U16.4 (AGND), U16.5 (PGND), U17.5 (GND), U17.7 (GND), U17.9 (GND), U18.6 (GND)
- net L: now also U18.5 (VA)
- net LB: now also U6.5 (PE6)
- net LG: now also U6.4 (PE5)
- net LR: now also U6.3 (PE4)
- net R: now also U18.8 (VB)
- net at U6.43 (PE12): now also U18.1 (SCK)
- net at U6.44 (PE13): now also U18.4 (SDO)
- net at U6.45 (PE14): now also U18.2 (SDI)
- net at U6.46 (PE15): now also U18.3 (~{CS}/LD)
- new net: R82.1, U16.7 (FA/SD)
- new net: R87.1, R88.2, U17.6 (FB)
- new net: D14.2 (A), L10.2, Q12.3 (D)
- new net: C91.2, D16.2 (A), D17.1 (K), R89.2
- new net: C83.2, C84.2, U16.2 (COMP)
- new net: C83.1, R81.2
- new net: Q12.2 (S), R83.2, R84.1
- new net: Q12.1 (G), U16.6 (DR)
- new net: C90.2, D15.1 (K), L11.1, U17.8 (SW)
- new net: C90.1, D16.1 (K), U17.1 (BOOST)
- new net +12V: J11.1 (Pin_1), L11.2, R87.2
- new net +15V: C88.1, C89.1, D14.1 (K), R85.2, R89.1, U17.2 (VIN), U17.3 (VCC), U17.4 (EN)
- new net FB_15: R85.1, R86.2, U16.3 (FB)
- new net ISEN_15: C86.2, R83.1, U16.1 (ISEN)

Commit message: file sync
Parts:
- added J12, J13: Conn_01x02_Male, symbol Connector:Conn_01x02_Male
- C67, C69, C70: footprint (none) -> Capacitor_SMD:C_0603_1608Metric
- C68, C72: footprint (none) -> Capacitor_SMD:C_0805_2012Metric
- C71: value 27uF -> 22uF; footprint (none) -> Capacitor_SMD:C_0805_2012Metric
- C73: value 4.7uF -> 1uF
- D17: value D_Zener_Small -> MMSZ5230BS
- F1: value 6V/5A -> F0603SB8000V032TM
Connections:
- net +12V: now also J12.1 (Pin_1), J13.1 (Pin_1)
- net GND: now also J12.2 (Pin_2), J13.2 (Pin_2)

Commit message: file sync
Parts:
- C73, C74, C76, C77, C78, C79, C80, C81, C82: footprint (none) -> Capacitor_SMD:C_0603_1608Metric
- C75: footprint (none) -> Capacitor_SMD:C_0805_2012Metric
- C88: footprint Capacitor_SMD:CP_Elec_6.3x5.9 -> Capacitor_SMD:C_0805_2012Metric
- D1, D2, D3, D4, D5: footprint (none) -> Diode_SMD:D_0603_1608Metric
- D10, D14, D9: footprint (none) -> Diode_SMD:D_SOD-123
- D11, D12, D17: footprint (none) -> Diode_SMD:D_SOD-323
- D13: footprint (none) -> Package_TO_SOT_SMD:SOT-23-3
- D15, D16, D8: footprint (none) -> Diode_SMD:D_SOD-523
- D6, D7: footprint (none) -> Diode_SMD:D_SOD-123F
- F1: footprint (none) -> Fuse:Fuse_0603_1608Metric
- J1: footprint (none) -> Footprints:TYPE-C-31-M-31
- J10, J11, J12, J13, J8, J9: footprint (none) -> Connector_PinSocket_2.54mm:PinSocket_1x02_P2.54mm_Vertical
- J2: footprint (none) -> Connector_Wire:SolderWire-1sqmm_1x02_P5.4mm_D1.4mm_OD2.7mm
- J3: footprint (none) -> Connector_PinHeader_2.00mm:PinHeader_1x04_P2.00mm_Vertical
- J4: footprint (none) -> Connector_PinHeader_2.00mm:PinHeader_1x18_P2.00mm_Vertical
- J5: footprint (none) -> Footprints:FCI_87520-0010BLF
- J6, J7: footprint (none) -> Connector_PinSocket_2.54mm:PinSocket_1x03_P2.54mm_Vertical
- L1: footprint (none) -> Inductor_SMD:L_12x12mm_H8mm
- L2: footprint (none) -> Footprints:L_0806_2016Metric
- L3: value BKW0805UCR12JST -> FNR6045S121MT; footprint (none) -> Inductor_SMD:L_6.3x6.3_H3
- L4: value BKW0805UCR12JST -> YPRH1207-151M

Commit message: schem complete
Parts:
- D13: footprint Package_TO_SOT_SMD:SOT-23-3 -> Package_TO_SOT_SMD:SOT-23
- L10: value BKW0805UCR12JST -> FNR6045S150MT; footprint (none) -> Inductor_SMD:L_6.3x6.3_H3
- L11: footprint (none) -> Inductor_SMD:L_1210_3225Metric
- L4: footprint (none) -> Inductor_SMD:L_12x12mm_H8mm
- L5: footprint (none) -> Inductor_SMD:L_1008_2520Metric
- L6: footprint (none) -> Inductor_SMD:L_0603_1608Metric
- L7, L8: value 15uH -> CBC3225T220KR; footprint (none) -> Inductor_SMD:L_1210_3225Metric
- L9: value 2.2uH -> DFE322512F-2R2M=P2; footprint (none) -> Resistor_SMD:R_1210_3225Metric
- Q1: footprint (none) -> Footprints:IRL7486MTRPbF
- Q12, Q7, Q8: footprint (none) -> Package_TO_SOT_SMD:SOT-23
- Q2, Q3: footprint (none) -> Footprints:PDFN3333-8
- Q4, Q5: footprint (none) -> Footprints:DFN-6L-2EP-2x2
- Q6: footprint (none) -> Package_TO_SOT_SMD:SOT-23-6
- R1, R11, R14, R15, R16, R17, R18, R19, R2, R20, R21, R22, R23, R24, R25, R26, R29, R3, R30, R31, R32, R35, R36, R37, R38, R39, R4, R40, R41, R42, R43, R44, R45, R46, R47, R48, R49, R5, R52, R53, R54, R55, R56, R57, R58, R59, R6, R60, R61, R62, R63, R64, R65, R66, R67, R68, R69, R7, R70, R71, R72, R73, R74, R75, R76, R77, R78, R79, R8, R80, R81, R82, R85, R86, R87, R88, R89, TH1: footprint (none) -> Resistor_SMD:R_0603_1608Metric
- R10, R13, R27, R28, R33, R34, R50, R51, R83, R84, Y2: footprint (none) -> Resistor_SMD:R_0805_2012Metric
- R12: footprint (none) -> Resistor_SMD:R_1206_3216Metric_Pad1.30x1.75mm_HandSolder
- R9: footprint (none) -> Resistor_SMD:R_1206_3216Metric
- RN1: footprint (none) -> Resistor_SMD:R_Array_Concave_4x0603
- TP1, TP2, TP3: footprint (none) -> TestPoint:TestPoint_Pad_1.0x1.0mm
- U1: footprint (none) -> Package_DFN_QFN:QFN-48-1EP_7x7mm_P0.5mm_EP5.3x5.3mm
- U10, U11: footprint (none) -> Package_SON:WSON-6-1EP_2x2mm_P0.65mm_EP1x1.6mm
- U14, U16, U17, U4, U5: footprint (none) -> Package_SO:VSSOP-8_3.0x3.0mm_P0.65mm
- U15: footprint (none) -> Package_SO:TSSOP-14_4.4x5mm_P0.65mm
- U18: footprint (none) -> Package_SO:SO-8_3.9x4.9mm_P1.27mm
- U3: footprint (none) -> Package_DFN_QFN:DFN-10-1EP_3x3mm_P0.5mm_EP1.65x2.38mm
- U7: footprint (none) -> Footprints:QFN-44_12x12_Pitch0.9mm
- U9: footprint DNP0006A -> Footprints:OPT3001DNPR
- Y1: footprint (none) -> Crystal:Crystal_SMD_2016-4Pin_2.0x1.6mm

Commit message: file sync
Connections:
- net at C10.2, L1.1, Q2.5 (D)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: now also Q2.1 (S), Q2.6 (D)
- net at Q2.7 (D), U1.15 (PCIN): now also Q2.8 (D), R10.1, R9.1
- net at C13.2, L1.2, Q3.5 (D)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: now also Q3.1 (S), Q3.6 (D)
- net at Q3.8 (D), R12.1, R13.1: now also Q3.7 (D), U1.24 (PCON)
Other:
- moved on the sheet: C12, C9, Q2B, Q3B, R10, R11, R13, R14
