File: VFDFFT.kicad_sch (KiCad schematic)
At the start: 261 parts, among them J1 USB_C_Receptacle_USB2.0, J10 Conn_01x02_Pin, J11 Conn_01x02_Male, J12 Conn_01x02_Male, J13 Conn_01x02_Male, J2 BATT, J3 FILAMENT+, J4 VFD_SIG, J5 USB_A, J6 Conn_01x03_Socket, J7 Conn_01x03_Socket, J8 Conn_01x02_Pin, J9 Conn_01x02_Pin, Q1 IRL7486MTRPBF, Q10 AO3400A, Q11 AO3400A, Q12 FS5N10S, Q2 ASDM30DN40E, Q3 ASDM30DN40E, Q4 HSCB2903, Q5 HSCB2903, Q6 AP6800, Q7 FS5N10S, Q8 FS5N10S, Q9 AO3400A, U1 IP2368, U10 TPS61170, U11 TPS61170, U12 W25Q128JVS, U13 TPS62170DSG, U14 LM358, U15 LM324, U16 LM3478, U17 LM2738, U18 LTC1446, U2 78L05_SOT23, U3 TPS40305, U4 LM3478, U5 LM3478, U6 STM32F446VETx, U7 AP6181, U8 HDC1080, U9 OPT3001DNPR, X1 SX1M32.768KM10F30TNN, Y1 26M, Y2 24M

Commit message: file sync
Parts:
- removed U18: LTC1446, Package_SO:SO-8_3.9x4.9mm_P1.27mm, symbol Analog_DAC:LTC1446
- removed Y1: 26M, Crystal:Crystal_SMD_2016-4Pin_2.0x1.6mm, symbol Device:Crystal_Small
- added C92, C93, C94: 1uF, Capacitor_SMD:C_0603_1608Metric, symbol Device:C_Small
- added C95: 10uF, Capacitor_SMD:C_0603_1608Metric, symbol Device:C_Small
- added C96, C97: 4.7uF, Capacitor_SMD:C_0603_1608Metric, symbol Device:C_Small
- added C98: 3.3nF, Capacitor_SMD:C_0603_1608Metric, symbol Device:C_Small
- added J14: AudioJack3_Ground, Footprints:TRRS-PJ-320A, symbol Connector_Audio:AudioJack3_Ground
- added J15: USB_C_Receptacle_USB2.0, Footprints:TYPE-C-31-M-31, symbol Connector:USB_C_Receptacle_USB2.0
- added R90, R91: 100K, Capacitor_SMD:C_0603_1608Metric, symbol Device:R_Small
- added R92, R93: 1K, Resistor_SMD:R_0603_1608Metric, symbol Device:R_Small
- added R94, R95: 5K1, Resistor_SMD:R_0603_1608Metric, symbol Device:R_Small
- added RN2: 22, Resistor_SMD:R_Array_Concave_4x0603, symbol Device:R_Pack04_Split
- added U18: ES9023, Package_SO:SO-16_3.9x9.9mm_P1.27mm, symbol Project_Symbols:ES9023
- added U19: CH340E, Package_SO:MSOP-10_3x3mm_P0.5mm, symbol Interface_USB:CH340E
- added Y1: WTL3M45404LZ, Crystal:Crystal_SMD_3225-4Pin_3.2x2.5mm, symbol Device:Crystal_GND24_Small
Connections:
- net DAC1 is gone; now on net L: U6.29 (PA4)
- net DAC2 is gone; now on net R: U6.30 (PA5)
- net +3V3: now also C94.1, R91.1, U18.5 (AVCC)
- net GND: now also C93.2, C94.2, C95.2, C96.2, C97.2, C98.2, J14.G, J14.S, J15.A1 (GND), J15.A12 (GND), J15.B1 (GND), J15.B12 (GND), J15.S1 (SHIELD), R90.2, R94.1, R95.1, U18.12 (AGND), U18.14 (DGND), U18.4 (DIF), U19.3 (GND), Y1.2, Y1.4
- net VFD_CLK: now also U6.43 (PE12); no longer U6.52 (PB13)
- net VFD_CS: now also U6.44 (PE13); no longer U6.15 (PC0)
- net VFD_DATA: now also U6.45 (PE14); no longer U6.16 (PC1)
- net VFD_RST: now also U6.46 (PE15); no longer U6.51 (PB12)
- net D-: now reaches J5.2 (D-), U6.53 (PB14)
- net D+: now reaches J5.3 (D+), U6.54 (PB15)
- net at C47.1, U7.10 (XTAL_IN): now also Y1.1; no longer C48.1
- net at R42.2: now also C48.1, Y1.3
- net AUX_MCK: now reaches U6.63 (PC6)
- net AUX_MCK: now also RN2.5 (R4.2)
- net at U6.68 (PA9): now also R92.1
- net at U6.69 (PA10): now also R93.1
- new net: C98.1, U19.10 (V3)
- new net: R93.2, U19.8 (TXD)
- new net: R92.2, U19.9 (RXD)
- new net: RN2.3 (R3.1), U18.1 (BCK)
- new net: C92.2, U18.10 (CN)
- new net: C93.1, U18.11 (NEG)
- new net: RN2.4 (R4.1), U18.13 (MCLK)
- new net: R91.2, U18.15 (MUTE_B)
- new net: RN2.2 (R2.1), U18.2 (LRCK)
- new net: RN2.1 (R1.1), U18.3 (SDI)
- new net: C95.1, R90.1, U18.6 (VREG)
- new net: C92.1, U18.9 (CP)
- new net: J15.A5 (CC1), R95.2
- new net: J15.B5 (CC2), R94.2
- new net AUX_I2S_CK: RN2.6 (R3.2), U6.52 (PB13)
- new net AUX_I2S_SD: RN2.8 (R1.2), U6.16 (PC1)
- new net AUX_I2S_WS: RN2.7 (R2.2), U6.51 (PB12)
- new net AUX_L: C96.1, J14.T, U18.7 (AOUTL)
- new net AUX_R: C97.1, J14.R, U18.8 (AOUTR)
- new net UD+: J15.A6 (D+), J15.B6 (D+), U19.1 (UD+)
- new net UD-: J15.A7 (D-), J15.B7 (D-), U19.2 (UD-)
- new net VBS: J15.A4 (VBUS), J15.A9 (VBUS), J15.B4 (VBUS), J15.B9 (VBUS), U19.7 (VCC)
- no-connect marks 23 -> 70

Commit message: file sync
Parts:
- removed Y2: 24M, Resistor_SMD:R_0805_2012Metric, symbol Device:Crystal_Small
- added Y2: 24M, Crystal:Crystal_SMD_3225-4Pin_3.2x2.5mm, symbol Device:Crystal_GND24_Small
- C65, C66: value 10nF -> ??
Connections:
- net GND: now also Y2.2, Y2.4
- net at C66.2, U6.13 (PH1): now also Y2.1
- net at C65.2, U6.12 (PH0): now also Y2.3
Changed lines of the file:
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@@
   (junction (at 58.42 175.26) (diameter 0) (color 0 0 0 0)
   )
+  (junction (at 293.37 78.74) (diameter 0) (color 0 0 0 0)
+  )
   (junction (at 104.775 25.4) (diameter 0) (color 0 0 0 0)
   )
@@
   (junction (at 168.275 269.875) (diameter 0) (color 0 0 0 0)
   )
+  (junction (at 283.845 78.74) (diameter 0) (color 0 0 0 0)
+  )
   (junction (at 40.005 97.79) (diameter 0) (color 0 0 0 0)
   )
@@
     (stroke (width 0) (type default))
   )
+  (wire (pts (xy 291.465 78.74) (xy 291.465 80.645))
+    (stroke (width 0) (type default))
+  )
   (wire (pts (xy 199.39 241.935) (xy 202.565 241.935))
     (stroke (width 0) (type default))
@@
     (stroke (width 0) (type default))
   )
+  (wire (pts (xy 290.83 78.74) (xy 288.925 78.74))
+    (stroke (width 0) (type default))
+  )
   (wire (pts (xy 169.545 239.395) (xy 190.5 239.395))
     (stroke (width 0) (type default))
@@
     (stroke (width 0) (type default))
   )
-  (wire (pts (xy 299.085 81.28) (xy 299.085 83.82))
+  (wire (pts (xy 299.085 81.28) (xy 299.085 84.455))
     (stroke (width 0) (type default))
   )
@@
     (stroke (width 0) (type default))
   )
+  (wire (pts (xy 297.18 83.82) (xy 297.18 78.74))
+    (stroke (width 0) (type default))
+  )
   (wire (pts (xy 64.135 99.695) (xy 64.135 100.33))
     (stroke (width 0) (type default))
@@
     (stroke (width 0) (type default))
   )
+  (wire (pts (xy 293.37 78.74) (xy 291.465 78.74))
+    (stroke (width 0) (type default))
+  )
   (wire (pts (xy 75.565 119.38) (xy 75.565 121.92))
     (stroke (width 0) (type default))
@@
     (stroke (width 0) (type default))
   )
+  (wire (pts (xy 293.37 83.82) (xy 297.18 83.82))
+    (stroke (width 0) (type default))
+  )
   (wire (pts (xy 210.82 168.91) (xy 210.82 169.545))
     (stroke (width 0) (type default))
   )
+  (wire (pts (xy 297.815 77.47) (xy 297.815 78.74))
+    (stroke (width 0) (type default))
+  )
   (wire (pts (xy 175.26 275.59) (xy 187.96 275.59))
     (stroke (width 0) (type default))
@@
     (stroke (width 0) (type default))
   )
-  (wire (pts (xy 290.83 83.82) (xy 290.83 82.55))
+  (wire (pts (xy 290.83 84.455) (xy 290.83 82.55))
     (stroke (width 0) (type default))
   )
@@
     (stroke (width 0) (type default))
   )
+  (wire (pts (xy 283.845 80.645) (xy 283.845 78.74))
+    (stroke (width 0) (type default))
+  )
   (wire (pts (xy 57.15 111.76) (xy 57.15 112.395))
     (stroke (width 0) (type default))
@@
     (stroke (width 0) (type default))
   )
-  (wire (pts (xy 288.925 78.74) (xy 297.815 78.74))
+  (wire (pts (xy 290.83 77.47) (xy 297.815 77.47))
     (stroke (width 0) (type default))
   )
@@
     (stroke (width 0) (type default))
   )
+  (wire (pts (xy 290.83 77.47) (xy 290.83 78.74))
+    (stroke (width 0) (type default))
+  )
   (wire (pts (xy 295.275 116.84) (xy 299.085 116.84))
     (stroke (width 0) (type default))
@@
     (stroke (width 0) (type default))
   )
+  (wire (pts (xy 297.18 78.74) (xy 293.37 78.74))
+    (stroke (width 0) (type default))
+  )
   (wire (pts (xy 73.66 252.73) (xy 73.66 264.16))
     (stroke (width 0) (type default))
@@
     (stroke (width 0) (type default))
   )
-  (wire (pts (xy 299.085 83.82) (xy 290.83 83.82))
+  (wire (pts (xy 299.085 84.455) (xy 290.83 84.455))
     (stroke (width 0) (type default))
   )
@@
     (stroke (width 0) (type default))
   )
+  (wire (pts (xy 291.465 80.645) (xy 283.845 80.645))
+    (stroke (width 0) (type default))
+  )
   (wire (pts (xy 179.07 62.23) (xy 182.245 62.23))
     (stroke (width 0) (type default))
@@
     )
   )
-  (symbol (lib_id "Device:Crystal_Small") (at 293.37 81.28 0) (unit 1)
-    (in_bom yes) (on_board yes) (dnp no)
-    (property "Reference" "Y2" (at 295.91 81.915 0)
-      (effects (font (size 0.8 0.8)))
-    )
-    (property "Value" "24M" (at 295.91 80.645 0)
-      (effects (font (size 0.8 0.8)))
-    )
-    (property "Footprint" "Resistor_SMD:R_0805_2012Metric" (at 293.37 81.28 0)
-      (effects (font (size 1.27 1.27)) hide)
-    )
-    (property "Datasheet" "~" (at 293.37 81.28 0)
-      (effects (font (size 1.27 1.27)) hide)
-    )
-    (pin "1")
-    (pin "2")
-    (instances
-      (project "VFDFFT"
-        (path "/7a53a631-dec5-4274-9a20-e8f914b63ed5"
-          (reference "Y2") (unit 1)
-        )
-      )
-    )
-  )
   (symbol (lib_id "power:GND") (at 91.44 116.205 180) (unit 1)
     (in_bom yes) (on_board yes) (dnp no) (fields_autoplaced)
@@
       (effects (font (size 0.8 0.8)) (justify left))
     )
-    (property "Value" "10nF" (at 290.195 81.915 90)
+    (property "Value" "??" (at 290.195 81.915 90)
       (effects (font (size 0.8 0.8)) (justify left))
     )
@@
       (effects (font (size 0.8 0.8)) (justify left))
     )
-    (property "Value" "10nF" (at 290.195 78.105 90)
+    (property "Value" "??" (at 290.195 78.105 90)
       (effects (font (size 0.8 0.8)) (justify left))
     )
@@
         )
       )
+    )
+  )
+  (symbol (lib_id "Device:Crystal_GND24_Small") (at 293.37 81.28 0) (unit 1)
+    (in_bom yes) (on_board yes) (dnp no)
+    (property "Reference" "Y2" (at 296.545 80.645 0)
+      (effects (font (size 0.8 0.8)))
+    )
+    (property "Value" "24M" (at 295.91 82.55 0)
+      (effects (font (size 0.8 0.8)))
+    )
+    (property "Footprint" "Crystal:Crystal_SMD_3225-4Pin_3.2x2.5mm" (at 293.37 81.28 0)
+      (effects (font (size 1.27 1.27)) hide)
+    )
+    (property "Datasheet" "~" (at 293.37 81.28 0)
+      (effects (font (size 1.27 1.27)) hide)
+    )
+    (pin "1")
+    (pin "2")
+    (pin "3")
+    (pin "4")
+    (instances
+      (project "VFDFFT"
+        (path "/7a53a631-dec5-4274-9a20-e8f914b63ed5"
+          (reference "Y2") (unit 1)
+        )
+      )

Commit message: Laser ON/OFF
Parts:
- removed J12, J13: Conn_01x02_Male, Connector_PinSocket_2.54mm:PinSocket_1x02_P2.54mm_Vertical, symbol Connector:Conn_01x02_Male
- J10, J11, J8, J9: footprint Connector_PinSocket_2.54mm:PinSocket_1x02_P2.54mm_Vertical -> Connector_PinSocket_2.00mm:PinSocket_1x02_P2.00mm_Vertical
Changed lines of the file:
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@@
     )
   )
-  (symbol (lib_id "power:GND") (at 122.555 200.66 90) (unit 1)
-    (in_bom yes) (on_board yes) (dnp no)
-    (property "Reference" "#PWR0285" (at 128.905 200.66 0)
-      (effects (font (size 1.27 1.27)) hide)
-    )
-    (property "Value" "GND" (at 122.555 201.295 90)
-      (effects (font (size 0.8 0.8)))
-    )
-    (property "Footprint" "" (at 122.555 200.66 0)
-      (effects (font (size 1.27 1.27)) hide)
-    )
-    (property "Datasheet" "" (at 122.555 200.66 0)
-      (effects (font (size 1.27 1.27)) hide)
-    )
-    (pin "1")
-    (instances
-      (project "VFDFFT"
-        (path "/7a53a631-dec5-4274-9a20-e8f914b63ed5"
-          (reference "#PWR0285") (unit 1)
-        )
-      )
-    )
-  )
   (symbol (lib_id "Device:D_TVS") (at 131.445 71.12 90) (mirror x) (unit 1)
     (in_bom yes) (on_board yes) (dnp no)
@@
       (effects (font (size 1.27 1.27)) (justify right))
     )
-    (property "Footprint" "Connector_PinSocket_2.54mm:PinSocket_1x02_P2.54mm_Vertical" (at 129.54 257.81 0)
+    (property "Footprint" "Connector_PinSocket_2.00mm:PinSocket_1x02_P2.00mm_Vertical" (at 129.54 257.81 0)
       (effects (font (size 1.27 1.27)) hide)
     )
@@
     )
   )
-  (symbol (lib_id "Connector:Conn_01x02_Male") (at 117.475 198.12 0) (unit 1)
-    (in_bom yes) (on_board yes) (dnp no) (fields_autoplaced)
-    (property "Reference" "J13" (at 118.11 193.675 0)
-      (effects (font (size 1.27 1.27)))
-    )
-    (property "Value" "Conn_01x02_Male" (at 118.11 196.215 0)
-      (effects (font (size 1.27 1.27)))
-    )
-    (property "Footprint" "Connector_PinSocket_2.54mm:PinSocket_1x02_P2.54mm_Vertical" (at 117.475 198.12 0)
-      (effects (font (size 1.27 1.27)) hide)
-    )
-    (property "Datasheet" "~" (at 117.475 198.12 0)
-      (effects (font (size 1.27 1.27)) hide)
-    )
-    (pin "1")
-    (pin "2")
-    (instances
-      (project "VFDFFT"
-        (path "/7a53a631-dec5-4274-9a20-e8f914b63ed5"
-          (reference "J13") (unit 1)
-        )
-      )
-    )
-  )
   (symbol (lib_id "Connector:Conn_01x02_Pin") (at 129.54 232.41 0) (mirror y) (unit 1)
     (in_bom yes) (on_board yes) (dnp no)
@@
       (effects (font (size 1.27 1.27)) (justify right))
     )
-    (property "Footprint" "Connector_PinSocket_2.54mm:PinSocket_1x02_P2.54mm_Vertical" (at 129.54 232.41 0)
+    (property "Footprint" "Connector_PinSocket_2.00mm:PinSocket_1x02_P2.00mm_Vertical" (at 129.54 232.41 0)
       (effects (font (size 1.27 1.27)) hide)
     )
@@
     )
   )
-  (symbol (lib_id "power:+12V") (at 122.555 187.325 270) (unit 1)
-    (in_bom yes) (on_board yes) (dnp no) (fields_autoplaced)
-    (property "Reference" "#PWR014" (at 118.745 187.325 0)
-      (effects (font (size 1.27 1.27)) hide)
-    )
-    (property "Value" "+12V" (at 126.365 187.96 90)
-      (effects (font (size 1.27 1.27)) (justify left))
-    )
-    (property "Footprint" "" (at 122.555 187.325 0)
-      (effects (font (size 1.27 1.27)) hide)
-    )
-    (property "Datasheet" "" (at 122.555 187.325 0)
-      (effects (font (size 1.27 1.27)) hide)
-    )
-    (pin "1")
-    (instances
-      (project "VFDFFT"
-        (path "/7a53a631-dec5-4274-9a20-e8f914b63ed5"
-          (reference "#PWR014") (unit 1)
-        )
-      )
-    )
-  )
   (symbol (lib_id "Device:R_Small") (at 78.105 83.185 270) (unit 1)
     (in_bom yes) (on_board yes) (dnp no)
@@
     )
   )
-  (symbol (lib_id "power:+12V") (at 122.555 198.12 270) (unit 1)
-    (in_bom yes) (on_board yes) (dnp no) (fields_autoplaced)
-    (property "Reference" "#PWR015" (at 118.745 198.12 0)
-      (effects (font (size 1.27 1.27)) hide)
-    )
-    (property "Value" "+12V" (at 126.365 198.755 90)
-      (effects (font (size 1.27 1.27)) (justify left))
-    )
-    (property "Footprint" "" (at 122.555 198.12 0)
-      (effects (font (size 1.27 1.27)) hide)
-    )
-    (property "Datasheet" "" (at 122.555 198.12 0)
-      (effects (font (size 1.27 1.27)) hide)
-    )
-    (pin "1")
-    (instances
-      (project "VFDFFT"
-        (path "/7a53a631-dec5-4274-9a20-e8f914b63ed5"
-          (reference "#PWR015") (unit 1)
-        )
-      )
-    )
-  )
   (symbol (lib_id "Device:C_Small") (at 67.31 65.405 0) (unit 1)
     (in_bom yes) (on_board yes) (dnp no)
@@
       (effects (font (size 1.27 1.27)))
     )
-    (property "Footprint" "Connector_PinSocket_2.54mm:PinSocket_1x02_P2.54mm_Vertical" (at 117.475 177.165 0)
+    (property "Footprint" "Connector_PinSocket_2.00mm:PinSocket_1x02_P2.00mm_Vertical" (at 117.475 177.165 0)
       (effects (font (size 1.27 1.27)) hide)
     )
@@
       (effects (font (size 1.27 1.27)) (justify right))
     )
-    (property "Footprint" "Connector_PinSocket_2.54mm:PinSocket_1x02_P2.54mm_Vertical" (at 129.54 245.11 0)
+    (property "Footprint" "Connector_PinSocket_2.00mm:PinSocket_1x02_P2.00mm_Vertical" (at 129.54 245.11 0)
       (effects (font (size 1.27 1.27)) hide)
     )
@@
     )
   )
-  (symbol (lib_id "power:GND") (at 122.555 189.865 90) (unit 1)
-    (in_bom yes) (on_board yes) (dnp no)
-    (property "Reference" "#PWR0284" (at 128.905 189.865 0)
-      (effects (font (size 1.27 1.27)) hide)
-    )
-    (property "Value" "GND" (at 122.555 190.5 90)
-      (effects (font (size 0.8 0.8)))
-    )
-    (property "Footprint" "" (at 122.555 189.865 0)
-      (effects (font (size 1.27 1.27)) hide)
-    )
-    (property "Datasheet" "" (at 122.555 189.865 0)
-      (effects (font (size 1.27 1.27)) hide)
-    )
-    (pin "1")
-    (instances
-      (project "VFDFFT"
-        (path "/7a53a631-dec5-4274-9a20-e8f914b63ed5"
-          (reference "#PWR0284") (unit 1)
-        )
-      )
-    )
-  )
   (symbol (lib_id "power:PRI_HI") (at 82.55 117.475 270) (unit 1)
     (in_bom yes) (on_board yes) (dnp no)
@@
         )
       )
-    )
-  )
-  (symbol (lib_id "Connector:Conn_01x02_Male") (at 117.475 187.325 0) (unit 1)
-    (in_bom yes) (on_board yes) (dnp no) (fields_autoplaced)
-    (property "Reference" "J12" (at 118.11 182.88 0)
-      (effects (font (size 1.27 1.27)))
-    )
-    (property "Value" "Conn_01x02_Male" (at 118.11 185.42 0)
-      (effects (font (size 1.27 1.27)))
-    )
-    (property "Footprint" "Connector_PinSocket_2.54mm:PinSocket_1x02_P2.54mm_Vertical" (at 117.475 187.325 0)
-      (effects (font (size 1.27 1.27)) hide)
-    )
-    (property "Datasheet" "~" (at 117.475 187.325 0)
-      (effects (font (size 1.27 1.27)) hide)
-    )
-    (pin "1")
-    (pin "2")
-    (instances
-      (project "VFDFFT"
-        (path "/7a53a631-dec5-4274-9a20-e8f914b63ed5"
-          (reference "J12") (unit 1)
-        )
-      )

Commit message: file sync
Parts:
- J6, J7: footprint Connector_PinSocket_2.54mm:PinSocket_1x03_P2.54mm_Vertical -> Connector_PinSocket_2.00mm:PinSocket_1x03_P2.00mm_Vertical
Changed lines of the file:
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@@
       (effects (font (size 1.27 1.27)) (justify left))
     )
-    (property "Footprint" "Connector_PinSocket_2.54mm:PinSocket_1x03_P2.54mm_Vertical" (at 335.915 243.205 0)
+    (property "Footprint" "Connector_PinSocket_2.00mm:PinSocket_1x03_P2.00mm_Vertical" (at 335.915 243.205 0)
       (effects (font (size 1.27 1.27)) hide)
     )
@@
       (effects (font (size 1.27 1.27)) (justify left))
     )
-    (property "Footprint" "Connector_PinSocket_2.54mm:PinSocket_1x03_P2.54mm_Vertical" (at 335.915 233.045 0)
+    (property "Footprint" "Connector_PinSocket_2.00mm:PinSocket_1x03_P2.00mm_Vertical" (at 335.915 233.045 0)
       (effects (font (size 1.27 1.27)) hide)
     )
