File: VFDFFT.kicad_sch (KiCad schematic)
At the start: 276 parts, among them J1 USB_C_Receptacle_USB2.0, J10 Conn_01x02_Pin, J11 Conn_01x02_Male, J14 AudioJack3_Ground, J15 USB_C_Receptacle_USB2.0, J2 BATT, J3 FILAMENT+, J4 VFD_SIG, J5 USB_A, J6 Conn_01x03_Socket, J7 Conn_01x03_Socket, J8 Conn_01x02_Pin, J9 Conn_01x02_Pin, Q1 IRL7486MTRPBF, Q10 AO3400A, Q11 AO3400A, Q12 FS5N10S, Q2 ASDM30DN40E, Q3 ASDM30DN40E, Q4 HSCB2903, Q5 HSCB2903, Q6 AP6800, Q7 FS5N10S, Q8 FS5N10S, Q9 AO3400A, U1 IP2368, U10 TPS61170, U11 TPS61170, U12 W25Q128JVS, U13 TPS62170DSG, U14 LM358, U15 LM324, U16 LM3478, U17 LM2738, U18 ES9023, U19 CH340E, U2 78L05_SOT23, U3 TPS40305, U4 LM3478, U5 LM3478, U6 STM32F446VETx, U7 AP6181, U8 HDC1080, U9 OPT3001DNPR, X1 SX1M32.768KM10F30TNN, Y1 TAXM26M4ZDBDDT2T, Y2 24M

Commit message: file sync
Parts:
- removed C42: 22uF, Capacitor_SMD:CP_Elec_6.3x5.9, symbol Device:C_Polarized_Small
- added C42, C99: 10uF, Capacitor_SMD:C_1210_3225Metric, symbol Device:C_Small
Connections:
- net GND: now also C42.2, C99.2
- net PRI_HI: now also C42.1, C99.1
Changed lines of the file:
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@@
   (junction (at 100.965 25.4) (diameter 0) (color 0 0 0 0)
   )
-  (junction (at 79.375 119.38) (diameter 0) (color 0 0 0 0)
-  )
   (junction (at 260.985 260.35) (diameter 0) (color 0 0 0 0)
   )
@@
   (junction (at 219.71 62.23) (diameter 0) (color 0 0 0 0)
   )
+  (junction (at 79.375 119.38) (diameter 0) (color 0 0 0 0)
+  )
   (junction (at 86.36 105.41) (diameter 0) (color 0 0 0 0)
   )
@@
     (stroke (width 0) (type default))
   )
+  (wire (pts (xy 79.375 119.38) (xy 83.185 119.38))
+    (stroke (width 0) (type default))
+  )
   (wire (pts (xy 40.005 97.155) (xy 40.005 97.79))
     (stroke (width 0) (type default))
@@
     )
   )
+  (symbol (lib_id "Device:C_Small") (at 83.185 121.92 0) (unit 1)
+    (in_bom yes) (on_board yes) (dnp no)
+    (property "Reference" "C99" (at 81.28 120.65 0)
+      (effects (font (size 0.8 0.8)) (justify left))
+    )
+    (property "Value" "10uF" (at 82.55 125.095 90)
+      (effects (font (size 0.8 0.8)) (justify left))
+    )
+    (property "Footprint" "Capacitor_SMD:C_1210_3225Metric" (at 83.185 121.92 0)
+      (effects (font (size 1.27 1.27)) hide)
+    )
+    (property "Datasheet" "~" (at 83.185 121.92 0)
+      (effects (font (size 1.27 1.27)) hide)
+    )
+    (pin "1")
+    (pin "2")
+    (instances
+      (project "VFDFFT"
+        (path "/7a53a631-dec5-4274-9a20-e8f914b63ed5"
+          (reference "C99") (unit 1)
+        )
+      )
+    )
+  )
   (symbol (lib_id "Device:Q_Dual_NMOS_S1G1D2S2G2D1") (at 55.88 94.615 0) (mirror y) (unit 1)
     (in_bom yes) (on_board yes) (dnp no)
@@
     )
   )
+  (symbol (lib_id "power:GND") (at 83.185 124.46 0) (unit 1)
+    (in_bom yes) (on_board yes) (dnp no) (fields_autoplaced)
+    (property "Reference" "#PWR0284" (at 83.185 130.81 0)
+      (effects (font (size 1.27 1.27)) hide)
+    )
+    (property "Value" "GND" (at 83.185 128.905 0)
+      (effects (font (size 1.27 1.27)) hide)
+    )
+    (property "Footprint" "" (at 83.185 124.46 0)
+      (effects (font (size 1.27 1.27)) hide)
+    )
+    (property "Datasheet" "" (at 83.185 124.46 0)
+      (effects (font (size 1.27 1.27)) hide)
+    )
+    (pin "1")
+    (instances
+      (project "VFDFFT"
+        (path "/7a53a631-dec5-4274-9a20-e8f914b63ed5"
+          (reference "#PWR0284") (unit 1)
+        )
+      )
+    )
+  )
   (symbol (lib_id "Device:C_Small") (at 149.225 85.725 0) (unit 1)
     (in_bom yes) (on_board yes) (dnp no)
@@
     )
   )
-  (symbol (lib_id "Device:C_Polarized_Small") (at 79.375 121.92 0) (unit 1)
-    (in_bom yes) (on_board yes) (dnp no)
-    (property "Reference" "C42" (at 79.375 120.65 0)
-      (effects (font (size 0.8 0.8)) (justify left))
-    )
-    (property "Value" "22uF" (at 79.375 123.19 0)
-      (effects (font (size 0.8 0.8)) (justify left))
-    )
-    (property "Footprint" "Capacitor_SMD:CP_Elec_6.3x5.9" (at 79.375 121.92 0)
-      (effects (font (size 1.27 1.27)) hide)
-    )
-    (property "Datasheet" "~" (at 79.375 121.92 0)
-      (effects (font (size 1.27 1.27)) hide)
-    )
-    (pin "1")
-    (pin "2")
-    (instances
-      (project "VFDFFT"
-        (path "/7a53a631-dec5-4274-9a20-e8f914b63ed5"
-          (reference "C42") (unit 1)
-        )
-      )
-    )
-  )
   (symbol (lib_id "power:GND") (at 124.46 127.635 90) (unit 1)
     (in_bom yes) (on_board yes) (dnp no) (fields_autoplaced)
@@
         )
       )
+    )
+  )
+  (symbol (lib_id "Device:C_Small") (at 79.375 121.92 0) (unit 1)
+    (in_bom yes) (on_board yes) (dnp no)
+    (property "Reference" "C42" (at 77.47 120.65 0)
+      (effects (font (size 0.8 0.8)) (justify left))
+    )
+    (property "Value" "10uF" (at 78.74 125.095 90)
+      (effects (font (size 0.8 0.8)) (justify left))
+    )
+    (property "Footprint" "Capacitor_SMD:C_1210_3225Metric" (at 79.375 121.92 0)
+      (effects (font (size 1.27 1.27)) hide)
+    )
+    (property "Datasheet" "~" (at 79.375 121.92 0)
+      (effects (font (size 1.27 1.27)) hide)
+    )
+    (pin "1")
+    (pin "2")
+    (instances
+      (project "VFDFFT"
+        (path "/7a53a631-dec5-4274-9a20-e8f914b63ed5"
+          (reference "C42") (unit 1)
+        )
+      )

Commit message: file sync
Parts:
- removed C36: 22uF, Capacitor_SMD:CP_Elec_6.3x5.9, symbol Device:C_Polarized_Small
- added C100, C101: 10uF, Capacitor_SMD:C_1210_3225Metric, symbol Device:C_Small
Connections:
- net GND: now also C100.2, C101.2
- net PRI_LO: now also C100.1
Changed lines of the file:
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@@
   (junction (at 57.15 142.24) (diameter 0) (color 0 0 0 0)
   )
-  (junction (at 79.375 144.145) (diameter 0) (color 0 0 0 0)
-  )
   (junction (at 98.425 237.49) (diameter 0) (color 0 0 0 0)
   )
@@
   (junction (at 235.585 137.16) (diameter 0) (color 0 0 0 0)
   )
+  (junction (at 79.375 144.145) (diameter 0) (color 0 0 0 0)
+  )
   (junction (at 168.91 250.19) (diameter 0) (color 0 0 0 0)
   )
@@
     )
   )
+  (symbol (lib_id "Device:C_Small") (at 79.375 146.685 0) (unit 1)
+    (in_bom yes) (on_board yes) (dnp no)
+    (property "Reference" "C100" (at 77.47 145.415 0)
+      (effects (font (size 0.8 0.8)) (justify left))
+    )
+    (property "Value" "10uF" (at 78.74 149.86 90)
+      (effects (font (size 0.8 0.8)) (justify left))
+    )
+    (property "Footprint" "Capacitor_SMD:C_1210_3225Metric" (at 79.375 146.685 0)
+      (effects (font (size 1.27 1.27)) hide)
+    )
+    (property "Datasheet" "~" (at 79.375 146.685 0)
+      (effects (font (size 1.27 1.27)) hide)
+    )
+    (pin "1")
+    (pin "2")
+    (instances
+      (project "VFDFFT"
+        (path "/7a53a631-dec5-4274-9a20-e8f914b63ed5"
+          (reference "C100") (unit 1)
+        )
+      )
+    )
+  )
   (symbol (lib_id "Device:C_Small") (at 91.44 105.41 90) (unit 1)
     (in_bom yes) (on_board yes) (dnp no)
@@
     )
   )
-  (symbol (lib_id "power:GND") (at 79.375 149.225 0) (unit 1)
-    (in_bom yes) (on_board yes) (dnp no) (fields_autoplaced)
-    (property "Reference" "#PWR0292" (at 79.375 155.575 0)
-      (effects (font (size 1.27 1.27)) hide)
-    )
-    (property "Value" "GND" (at 79.375 153.67 0)
-      (effects (font (size 1.27 1.27)) hide)
-    )
-    (property "Footprint" "" (at 79.375 149.225 0)
-      (effects (font (size 1.27 1.27)) hide)
-    )
-    (property "Datasheet" "" (at 79.375 149.225 0)
-      (effects (font (size 1.27 1.27)) hide)
-    )
-    (pin "1")
-    (instances
-      (project "VFDFFT"
-        (path "/7a53a631-dec5-4274-9a20-e8f914b63ed5"
-          (reference "#PWR0292") (unit 1)
-        )
-      )
-    )
-  )
   (symbol (lib_id "power:GND") (at 53.34 152.4 270) (unit 1)
     (in_bom yes) (on_board yes) (dnp no) (fields_autoplaced)
@@
     )
   )
-  (symbol (lib_id "Device:C_Polarized_Small") (at 79.375 146.685 0) (unit 1)
-    (in_bom yes) (on_board yes) (dnp no)
-    (property "Reference" "C36" (at 79.375 145.415 0)
-      (effects (font (size 0.8 0.8)) (justify left))
-    )
-    (property "Value" "22uF" (at 79.375 147.955 0)
-      (effects (font (size 0.8 0.8)) (justify left))
-    )
-    (property "Footprint" "Capacitor_SMD:CP_Elec_6.3x5.9" (at 79.375 146.685 0)
-      (effects (font (size 1.27 1.27)) hide)
-    )
-    (property "Datasheet" "~" (at 79.375 146.685 0)
-      (effects (font (size 1.27 1.27)) hide)
-    )
-    (pin "1")
-    (pin "2")
-    (instances
-      (project "VFDFFT"
-        (path "/7a53a631-dec5-4274-9a20-e8f914b63ed5"
-          (reference "C36") (unit 1)
-        )
-      )
-    )
-  )
   (symbol (lib_id "Device:C_Polarized_Small") (at 56.515 201.93 180) (unit 1)
     (in_bom yes) (on_board yes) (dnp no)
@@
     )
   )
+  (symbol (lib_id "power:GND") (at 79.375 149.225 0) (unit 1)
+    (in_bom yes) (on_board yes) (dnp no) (fields_autoplaced)
+    (property "Reference" "#PWR0285" (at 79.375 155.575 0)
+      (effects (font (size 1.27 1.27)) hide)
+    )
+    (property "Value" "GND" (at 79.375 153.67 0)
+      (effects (font (size 1.27 1.27)) hide)
+    )
+    (property "Footprint" "" (at 79.375 149.225 0)
+      (effects (font (size 1.27 1.27)) hide)
+    )
+    (property "Datasheet" "" (at 79.375 149.225 0)
+      (effects (font (size 1.27 1.27)) hide)
+    )
+    (pin "1")
+    (instances
+      (project "VFDFFT"
+        (path "/7a53a631-dec5-4274-9a20-e8f914b63ed5"
+          (reference "#PWR0285") (unit 1)
+        )
+      )
+    )
+  )
   (symbol (lib_id "power:GND") (at 131.445 37.465 90) (unit 1)
     (in_bom yes) (on_board yes) (dnp no)
@@
     )
   )
+  (symbol (lib_id "power:GND") (at 83.185 149.225 0) (unit 1)
+    (in_bom yes) (on_board yes) (dnp no) (fields_autoplaced)
+    (property "Reference" "#PWR0292" (at 83.185 155.575 0)
+      (effects (font (size 1.27 1.27)) hide)
+    )
+    (property "Value" "GND" (at 83.185 153.67 0)
+      (effects (font (size 1.27 1.27)) hide)
+    )
+    (property "Footprint" "" (at 83.185 149.225 0)
+      (effects (font (size 1.27 1.27)) hide)
+    )
+    (property "Datasheet" "" (at 83.185 149.225 0)
+      (effects (font (size 1.27 1.27)) hide)
+    )
+    (pin "1")
+    (instances
+      (project "VFDFFT"
+        (path "/7a53a631-dec5-4274-9a20-e8f914b63ed5"
+          (reference "#PWR0292") (unit 1)
+        )
+      )
+    )
+  )
   (symbol (lib_id "Device:R_Small") (at 240.665 241.3 270) (unit 1)
     (in_bom yes) (on_board yes) (dnp no)
@@
         )
       )
+    )
+  )
+  (symbol (lib_id "Device:C_Small") (at 83.185 146.685 0) (unit 1)
+    (in_bom yes) (on_board yes) (dnp no)
+    (property "Reference" "C101" (at 81.28 145.415 0)
+      (effects (font (size 0.8 0.8)) (justify left))
+    )
+    (property "Value" "10uF" (at 82.55 149.86 90)
+      (effects (font (size 0.8 0.8)) (justify left))
+    )
+    (property "Footprint" "Capacitor_SMD:C_1210_3225Metric" (at 83.185 146.685 0)
+      (effects (font (size 1.27 1.27)) hide)
+    )
+    (property "Datasheet" "~" (at 83.185 146.685 0)
+      (effects (font (size 1.27 1.27)) hide)
+    )
+    (pin "1")
+    (pin "2")
+    (instances
+      (project "VFDFFT"
+        (path "/7a53a631-dec5-4274-9a20-e8f914b63ed5"
+          (reference "C101") (unit 1)
+        )
+      )

Commit message: Lasesr GPIO
Connections:
- net LB: now also U6.57 (PD10); no longer U6.5 (PE6)
- net LG: now also U6.56 (PD9); no longer U6.4 (PE5)
- net LR: now also U6.55 (PD8); no longer U6.3 (PE4)
Changed lines of the file:
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@@
   (no_connect (at 179.705 33.02))
   (no_connect (at 208.28 169.545))
+  (no_connect (at 299.085 96.52))
   (no_connect (at 359.41 63.5))
   (no_connect (at 82.55 42.545))
@@
   (no_connect (at 344.805 165.1))
   (no_connect (at 299.085 142.24))
+  (no_connect (at 299.085 101.6))
   (no_connect (at 344.805 73.66))
   (no_connect (at 299.085 139.7))
   (no_connect (at 344.805 99.06))
-  (no_connect (at 299.085 152.4))
   (no_connect (at 299.085 104.14))
   (no_connect (at 344.805 147.32))
@@
   (no_connect (at 182.245 72.39))
   (no_connect (at 344.805 106.68))
+  (no_connect (at 299.085 99.06))
   (no_connect (at 359.41 50.8))
   (no_connect (at 44.45 54.61))
@@
   (no_connect (at 201.93 128.905))
   (no_connect (at 344.805 139.7))
-  (no_connect (at 299.085 154.94))
   (no_connect (at 299.085 144.78))
   (no_connect (at 82.55 50.165))
@@
   (no_connect (at 256.54 124.46))
   (no_connect (at 97.155 31.115))
-  (no_connect (at 299.085 149.86))
   (wire (pts (xy 84.455 82.55) (xy 84.455 83.185))
     (stroke (width 0) (type default))
@@
     (stroke (width 0) (type default))
   )
+  (wire (pts (xy 295.91 154.94) (xy 299.085 154.94))
+    (stroke (width 0) (type default))
+  )
   (wire (pts (xy 289.56 235.585) (xy 290.195 235.585))
     (stroke (width 0) (type default))
@@
     (stroke (width 0) (type default))
   )
+  (wire (pts (xy 295.91 149.86) (xy 299.085 149.86))
+    (stroke (width 0) (type default))
+  )
   (wire (pts (xy 127 81.915) (xy 127 83.185))
     (stroke (width 0) (type default))
@@
     (stroke (width 0) (type default))
   )
-  (wire (pts (xy 295.91 99.06) (xy 299.085 99.06))
-    (stroke (width 0) (type default))
-  )
   (wire (pts (xy 293.37 83.82) (xy 297.18 83.82))
     (stroke (width 0) (type default))
@@
     (stroke (width 0) (type default))
   )
+  (wire (pts (xy 295.91 152.4) (xy 299.085 152.4))
+    (stroke (width 0) (type default))
+  )
   (wire (pts (xy 237.49 139.7) (xy 241.3 139.7))
     (stroke (width 0) (type default))
@@
     (stroke (width 0) (type default))
   )
-  (wire (pts (xy 295.91 96.52) (xy 299.085 96.52))
-    (stroke (width 0) (type default))
-  )
   (wire (pts (xy 240.03 165.735) (xy 243.84 165.735))
     (stroke (width 0) (type default))
@@
   )
   (wire (pts (xy 207.645 125.73) (xy 219.075 125.73))
-    (stroke (width 0) (type default))
-  )
-  (wire (pts (xy 295.91 101.6) (xy 299.085 101.6))
     (stroke (width 0) (type default))
   )
@@
     (effects (font (size 0.8 0.8)) (justify left bottom))
   )
-  (label "LB" (at 295.91 101.6 0) (fields_autoplaced)
-    (effects (font (size 1.27 1.27)) (justify left bottom))
-  )
   (label "WL_HOST_WAKE" (at 217.17 67.31 180) (fields_autoplaced)
     (effects (font (size 0.8 0.8)) (justify right bottom))
@@
     (effects (font (size 1.27 1.27)) (justify right bottom))
   )
-  (label "LR" (at 295.91 96.52 0) (fields_autoplaced)
+  (label "LB" (at 295.91 154.94 0) (fields_autoplaced)
     (effects (font (size 1.27 1.27)) (justify left bottom))
   )
@@
     (effects (font (size 1.27 1.27)) (justify left bottom))
   )
+  (label "LG" (at 295.91 152.4 0) (fields_autoplaced)
+    (effects (font (size 1.27 1.27)) (justify left bottom))
+  )
   (label "WL_D3" (at 348.615 157.48 180) (fields_autoplaced)
     (effects (font (size 0.8 0.8)) (justify right bottom))
@@
   (label "WL_REG_ON" (at 215.265 64.77 180) (fields_autoplaced)
     (effects (font (size 0.8 0.8)) (justify right bottom))
-  )
-  (label "LG" (at 295.91 99.06 0) (fields_autoplaced)
-    (effects (font (size 1.27 1.27)) (justify left bottom))
   )
   (label "3v3_PG" (at 60.325 189.23 90) (fields_autoplaced)
@@
     (effects (font (size 1.27 1.27)) (justify right bottom))
   )
+  (label "LR" (at 295.91 149.86 0) (fields_autoplaced)
+    (effects (font (size 1.27 1.27)) (justify left bottom))
+  )
   (label "DP" (at 112.395 29.21 270) (fields_autoplaced)

Commit message: file sync
Parts:
- added X2: 12.288MHz, Crystal:Crystal_SMD_2016-4Pin_2.0x1.6mm, symbol Oscillator:IQXO-70
Connections:
- net +3V3: now also X2.4 (V+)
- net GND: now also X2.2 (GND)
- net HUM_SCK: now also U6.95 (PB8); no longer U6.67 (PA8)
- net HUM_SDA: now also U6.93 (PB7); no longer U6.66 (PC9)
- new net: U6.66 (PC9), X2.3 (OUT)
Changed lines of the file:
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@@
   (junction (at 87.63 180.34) (diameter 0) (color 0 0 0 0)
   )
+  (no_connect (at 371.475 152.4))
   (no_connect (at 381 73.66))
   (no_connect (at 205.74 169.545))
@@
   (no_connect (at 82.55 42.545))
   (no_connect (at 125.095 50.165))
-  (no_connect (at 344.805 109.22))
   (no_connect (at 344.805 111.76))
   (no_connect (at 299.085 129.54))
@@
   (no_connect (at 344.805 53.34))
   (no_connect (at 182.245 72.39))
-  (no_connect (at 344.805 106.68))
   (no_connect (at 299.085 99.06))
   (no_connect (at 359.41 50.8))
@@
   (no_connect (at 201.93 128.905))
   (no_connect (at 344.805 139.7))
+  (no_connect (at 344.805 66.04))
   (no_connect (at 299.085 144.78))
   (no_connect (at 82.55 50.165))
@@
     (stroke (width 0) (type default))
   )
+  (wire (pts (xy 344.805 152.4) (xy 356.235 152.4))
+    (stroke (width 0) (type default))
+  )
   (wire (pts (xy 216.535 64.135) (xy 220.98 64.135))
     (stroke (width 0) (type default))
@@
     (stroke (width 0) (type default))
   )
+  (wire (pts (xy 344.805 106.68) (xy 349.25 106.68))
+    (stroke (width 0) (type default))
+  )
   (wire (pts (xy 207.645 125.73) (xy 219.075 125.73))
     (stroke (width 0) (type default))
@@
     (stroke (width 0) (type default))
   )
-  (wire (pts (xy 348.615 152.4) (xy 344.805 152.4))
-    (stroke (width 0) (type default))
-  )
   (wire (pts (xy 295.91 81.28) (xy 297.815 81.28))
     (stroke (width 0) (type default))
@@
     (stroke (width 0) (type default))
   )
-  (wire (pts (xy 349.25 66.04) (xy 344.805 66.04))
+  (wire (pts (xy 349.25 109.22) (xy 344.805 109.22))
     (stroke (width 0) (type default))
   )
@@
     (effects (font (size 0.8 0.8)) (justify left bottom))
   )
-  (label "HUM_SDA" (at 348.615 152.4 180) (fields_autoplaced)
-    (effects (font (size 0.8 0.8)) (justify right bottom))
-  )
   (label "L-" (at 328.93 235.585 0) (fields_autoplaced)
     (effects (font (size 1.27 1.27)) (justify left bottom))
@@
     (effects (font (size 0.8 0.8)) (justify right bottom))
   )
+  (label "HUM_SDA" (at 349.25 106.68 180) (fields_autoplaced)
+    (effects (font (size 0.8 0.8)) (justify right bottom))
+  )
   (label "R+" (at 328.93 240.665 0) (fields_autoplaced)
     (effects (font (size 1.27 1.27)) (justify left bottom))
@@
     (effects (font (size 1.27 1.27)) (justify right bottom))
   )
-  (label "HUM_SCK" (at 349.25 66.04 180) (fields_autoplaced)
+  (label "HUM_SCK" (at 349.25 109.22 180) (fields_autoplaced)
     (effects (font (size 0.8 0.8)) (justify right bottom))
   )
@@
     )
   )
+  (symbol (lib_id "Oscillator:IQXO-70") (at 363.855 152.4 180) (unit 1)
+    (in_bom yes) (on_board yes) (dnp no) (fields_autoplaced)
+    (property "Reference" "X2" (at 372.11 147.3823 0)
+      (effects (font (size 1.27 1.27)))
+    )
+    (property "Value" "12.288MHz" (at 372.11 149.9223 0)
+      (effects (font (size 0.8 0.8)))
+    )
+    (property "Footprint" "Crystal:Crystal_SMD_2016-4Pin_2.0x1.6mm" (at 346.71 144.145 0)
+      (effects (font (size 1.27 1.27)) hide)
+    )
+    (property "Datasheet" "http://www.iqdfrequencyproducts.com/products/details/iqxo-70-11-30.pdf" (at 366.395 152.4 0)
+      (effects (font (size 1.27 1.27)) hide)
+    )
+    (pin "1")
+    (pin "2")
+    (pin "3")
+    (pin "4")
+    (instances
+      (project "VFDFFT"
+        (path "/7a53a631-dec5-4274-9a20-e8f914b63ed5"
+          (reference "X2") (unit 1)
+        )
+      )
+    )
+  )
   (symbol (lib_id "Connector:USB_C_Receptacle_USB2.0") (at 396.24 60.96 0) (mirror y) (unit 1)
     (in_bom yes) (on_board yes) (dnp no) (fields_autoplaced)
@@
     )
   )
+  (symbol (lib_id "power:GND") (at 363.855 144.78 180) (unit 1)
+    (in_bom yes) (on_board yes) (dnp no) (fields_autoplaced)
+    (property "Reference" "#PWR015" (at 363.855 138.43 0)
+      (effects (font (size 1.27 1.27)) hide)
+    )
+    (property "Value" "GND" (at 363.855 139.7 0)
+      (effects (font (size 1.27 1.27)) hide)
+    )
+    (property "Footprint" "" (at 363.855 144.78 0)
+      (effects (font (size 1.27 1.27)) hide)
+    )
+    (property "Datasheet" "" (at 363.855 144.78 0)
+      (effects (font (size 1.27 1.27)) hide)
+    )
+    (pin "1")
+    (instances
+      (project "VFDFFT"
+        (path "/7a53a631-dec5-4274-9a20-e8f914b63ed5"
+          (reference "#PWR015") (unit 1)
+        )
+      )
+    )
+  )
   (symbol (lib_id "power:GND") (at 133.35 67.31 90) (mirror x) (unit 1)
     (in_bom yes) (on_board yes) (dnp no)
@@
         )
       )
+    )
+  )
+  (symbol (lib_id "power:+3V3") (at 363.855 160.02 180) (unit 1)
+    (in_bom yes) (on_board yes) (dnp no)
+    (property "Reference" "#PWR014" (at 363.855 156.21 0)
+      (effects (font (size 1.27 1.27)) hide)
+    )
+    (property "Value" "+3V3" (at 364.49 159.385 90)
+      (effects (font (size 0.8 0.8)))
+    )
+    (property "Footprint" "" (at 363.855 160.02 0)
+      (effects (font (size 1.27 1.27)) hide)
+    )
+    (property "Datasheet" "" (at 363.855 160.02 0)
+      (effects (font (size 1.27 1.27)) hide)
+    )
+    (pin "1")
+    (instances
+      (project "VFDFFT"
+        (path "/7a53a631-dec5-4274-9a20-e8f914b63ed5"
+          (reference "#PWR014") (unit 1)
+        )
+      )

Commit message: file sync
Connections:
- net PRI_LO: now also C101.1
Changed lines of the file:
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@@
   (junction (at 63.5 62.865) (diameter 0) (color 0 0 0 0)
   )
+  (junction (at 83.185 142.24) (diameter 0) (color 0 0 0 0)
+  )
   (junction (at 27.94 205.74) (diameter 0) (color 0 0 0 0)
   )
@@
     (stroke (width 0) (type default))
   )
-  (wire (pts (xy 79.375 142.24) (xy 82.55 142.24))
+  (wire (pts (xy 79.375 142.24) (xy 83.185 142.24))
     (stroke (width 0) (type default))
   )
@@
     (stroke (width 0) (type default))
   )
+  (wire (pts (xy 83.185 142.24) (xy 83.185 144.145))
+    (stroke (width 0) (type default))
+  )
   (wire (pts (xy 63.5 62.865) (xy 67.31 62.865))
     (stroke (width 0) (type default))
@@
     )
   )
-  (symbol (lib_id "power:PRI_LO") (at 82.55 142.24 270) (unit 1)
+  (symbol (lib_id "power:PRI_LO") (at 83.185 142.24 270) (unit 1)
     (in_bom yes) (on_board yes) (dnp no)
-    (property "Reference" "#PWR0172" (at 78.74 142.24 0)
+    (property "Reference" "#PWR0172" (at 79.375 142.24 0)
       (effects (font (size 1.27 1.27)) hide)
     )
-    (property "Value" "PRI_LO" (at 79.375 141.605 90)
+    (property "Value" "PRI_LO" (at 80.01 141.605 90)
       (effects (font (size 0.8 0.8)) (justify left))
     )
-    (property "Footprint" "" (at 82.55 142.24 0)
+    (property "Footprint" "" (at 83.185 142.24 0)
       (effects (font (size 1.27 1.27)) hide)
     )
-    (property "Datasheet" "" (at 82.55 142.24 0)
+    (property "Datasheet" "" (at 83.185 142.24 0)
       (effects (font (size 1.27 1.27)) hide)
     )
