File: _autosave-VFDFFT.kicad_pcb (KiCad board)
At the start: 2 copper layers, 100 x 50 mm, 276 parts, among them J1 USB_C_Receptacle_USB2.0, J10 Conn_01x02_Pin, J11 Conn_01x02_Male, J14 AudioJack3_Ground, J15 USB_C_Receptacle_USB2.0, J2 BATT, J3 FILAMENT+, J4 VFD_SIG, J5 USB_A, J6 Conn_01x03_Socket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

Commit message: file sync
Other:
- board text added: "Charging Only No Data Here"
