File: VFDFFT.kicad_pcb (KiCad board)
At the start: 2 copper layers, 100 x 50 mm, 276 parts, among them J1 USB_C_Receptacle_USB2.0, J10 Conn_01x02_Pin, J11 Conn_01x02_Male, J14 AudioJack3_Ground, J15 USB_C_Receptacle_USB2.0, J2 BATT, J3 FILAMENT+, J4 VFD_SIG, J5 USB_A, J6 Conn_01x03_Socket, J7 Conn_01x03_Socket, J8 Conn_01x02_Pin, J9 Conn_01x02_Pin, Q1 IRL7486MTRPBF, Q10 AO3400A, Q11 AO3400A, Q12 FS5N10S, Q2 ASDM30DN40E, Q3 ASDM30DN40E, Q4 HSCB2903, Q5 HSCB2903, Q6 AP6800, Q7 FS5N10S, Q8 FS5N10S, Q9 AO3400A, U1 IP2368, U10 TPS61170, U11 TPS61170, U12 W25Q128JVS, U13 TPS62170DSG, U14 LM358, U15 LM324, U16 LM3478, U17 LM2738, U18 ES9023, U19 CH340E, U2 78L05_SOT23, U3 TPS40305, U4 LM3478, U5 LM3478, U6 STM32F446VETx, U7 AP6181, U8 HDC1080, U9 OPT3001DNPR, X1 SX1M32.768KM10F30TNN, Y1 TAXM26M4ZDBDDT2T, Y2 24M

Commit message: file sync
Parts:
- added C99: 10uF, Capacitor_SMD:C_1210_3225Metric, F.Cu at (122.4, 37.3)
- C42: value 22uF -> 10uF; footprint Capacitor_SMD:CP_Elec_6.3x5.9 -> Capacitor_SMD:C_1210_3225Metric
- moved C34 124.8 mm to (100.1, 21.9)
- moved C35 124.8 mm to (100.1, 24.4)
- moved C31 124.8 mm to (104.5, 9.85)
- moved C32 124.8 mm to (100.1, 16.9)
- moved C33 124.8 mm to (100.1, 19.4)
- moved C36 124.8 mm to (94.8, 11.6)
- moved D9 124.8 mm to (103.0, 13.9)
- moved L3 124.8 mm to (93.8, 19.6)
- moved Q7 124.8 mm to (108.5, 17.9)
- moved R25 124.8 mm to (100.1, 26.9)
- moved R26 124.8 mm to (104.1, 16.9)
- moved R27 124.8 mm to (104.1, 19.4)
- moved R30 124.8 mm to (104.1, 26.9)
- moved R28 124.8 mm to (104.1, 21.9)
- moved R29 124.8 mm to (104.1, 24.4)
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Routing:
- net +3V3: track 41.7 -> 155.0 mm, vias 0 -> 6
- net +BATT: track 80.6 -> 142.0 mm, vias 5 -> 9
- net GND: track 72.9 -> 125.2 mm, vias 55 -> 118
- net PRI_HI: track 0.00 -> 51.0 mm, vias 0 -> 2
- net /D-: track 0.00 -> 48.5 mm, vias 0 -> 1
- net /D+: track 0.00 -> 47.7 mm, vias 0 -> 1
- net /WL_D1: track 0.00 -> 41.5 mm, vias 0 -> 2
- net /WL_D2: track 0.00 -> 39.5 mm, vias 0 -> 2
- net /WL_CMD: track 0.00 -> 38.6 mm, vias 0 -> 2
- net /WL_D3: track 0.00 -> 38.2 mm, vias 0 -> 2
- net /WL_D0: track 0.00 -> 36.3 mm, vias 0 -> 2
- net /WL_CLK: track 0.00 -> 35.4 mm, vias 0 -> 2
- net /FLASH_IO0: track 0.00 -> 32.1 mm, vias 0 -> 2
- net /FLASH_SCK: track 0.00 -> 27.7 mm, vias 0 -> 2
- net /FLASH_IO1: track 0.00 -> 27.6 mm, vias 0 -> 2
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- added copper zone on F.Cu, net GND
Other:
- board text added: "Charging Only No Data Here"
- board text added: "装不回去了吧"

Commit message: file sync
Parts:
- removed C36: 22uF, Capacitor_SMD:CP_Elec_6.3x5.9
- added C100: 10uF, Capacitor_SMD:C_1210_3225Metric, F.Cu at (108.7, 48.0)
- added C101: 10uF, Capacitor_SMD:C_1210_3225Metric, F.Cu at (108.7, 52.8)
- D9: footprint Diode_SMD:D_1206_3216Metric -> Footprints:SOD-323HE
- moved R60 109.9 mm to (45.7, 75.2), turned to 180 degrees
- moved R59 106.8 mm to (48.8, 75.2), turned to 180 degrees
- moved L9 106.6 mm to (53.3, 73.6), turned to 90 degrees
- moved C78 104.4 mm to (51.1, 74.4), turned to -90 degrees
- moved U13 103.3 mm to (56.4, 74.4), turned to 180 degrees
- moved RN2 100.3 mm to (64.3, 62.2), turned to 90 degrees
- moved R61 99.7 mm to (56.4, 72.4)
- moved C77 96.6 mm to (58.9, 74.7), turned to -90 degrees
- moved D12 86.0 mm to (104.9, 39.9)
- moved R57 85.6 mm to (102.4, 43.9), turned to -90 degrees
- moved D11 84.3 mm to (101.6, 56.1), turned to 90 degrees
- moved R55 84.2 mm to (102.4, 40.9), turned to -90 degrees
- moved U11 84.2 mm to (103.5, 46.9), turned to 90 degrees
- moved U10 83.5 mm to (104.0, 55.8), turned to 90 degrees
- moved L7 83.2 mm to (103.6, 52.1), turned to -90 degrees
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Routing:
- net +BATT: track 142.0 -> 314.4 mm, vias 9 -> 17
- net +3V3: track 155.0 -> 257.1 mm, vias 6 -> 9
- net GNDA: track 0.00 -> 89.7 mm, vias 0 -> 7
- net GND: track 125.2 -> 193.8 mm, vias 118 -> 153
- net /OPT_SCL: track 6.87 -> 53.3 mm, vias 0 -> 2
- net VDDA: track 0.00 -> 46.2 mm, vias 0 -> 7
- net Net-(RN2D-R4.1): track 0.00 -> 33.9 mm, vias 0 -> 2
- net Net-(RN2A-R1.1): track 0.00 -> 31.6 mm, vias 0 -> 2
- net PRI_LO: track 0.00 -> 30.7 mm, vias 0 -> 2
- net Net-(RN2B-R2.1): track 0.00 -> 30.0 mm, vias 0 -> 2
- net Net-(RN2C-R3.1): track 0.00 -> 29.9 mm, vias 0 -> 2
- net /OPT_SDA: track 4.27 -> 31.4 mm, vias 0 -> 2
- net /AUX_I2S_SD: track 0.00 -> 25.0 mm, vias 0 -> 2
- net /FLASH_CS: track 2.09 -> 26.2 mm, vias 0 -> 2
- net /AUX_I2S_WS: track 0.00 -> 20.7 mm, vias 0 -> 2
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
Commit message: file sync
Parts:
- moved J6 45.1 mm to (93.0, 53.3), turned to 90 degrees
- moved J7 44.6 mm to (85.9, 53.8)
- moved R65 23.5 mm to (83.1, 49.0)
Routing:
- net GNDA: track 89.7 -> 105.6 mm
- net /R-: track 15.5 -> 30.3 mm, vias 2 -> 3
- net /R+: track 7.91 -> 16.6 mm
- net Net-(U15A--): track 10.5 -> 12.7 mm

Commit message: Lasesr GPIO
Parts:
- D9: footprint Footprints:SOD-323HE -> Diode_SMD:D_1206_3216Metric
- moved Q11 84.9 mm to (50.0, 46.0), turned to 90 degrees
- moved R80 82.5 mm to (47.5, 46.2), turned to -90 degrees
- moved R79 81.4 mm to (48.5, 43.2)
- moved Q10 81.3 mm to (55.1, 46.0), turned to 90 degrees
- moved R78 78.9 mm to (52.6, 46.2), turned to -90 degrees
- moved Q9 78.2 mm to (60.2, 46.0), turned to 90 degrees
- moved R77 77.8 mm to (53.6, 43.2)
- moved R75 76.9 mm to (57.7, 46.2), turned to -90 degrees
- moved J10 72.8 mm to (50.0, 40.6), turned to 90 degrees
- moved R76 72.4 mm to (60.2, 43.2)
- moved J9 68.4 mm to (55.9, 40.6), turned to 90 degrees
- moved J8 65.0 mm to (61.7, 40.6), turned to 90 degrees
Connections:
- C101 pad 1: PRI_LO -> unconnected-(C101-Pad1)
- U6 pad 3: /LR -> unconnected-(U6-PE4-Pad3)
- U6 pad 4: /LG -> unconnected-(U6-PE5-Pad4)
- U6 pad 5: /LB -> unconnected-(U6-PE6-Pad5)
- U6 pad 55: unconnected-(U6-PD8-Pad55) -> /LR
- U6 pad 56: unconnected-(U6-PD9-Pad56) -> /LG
- U6 pad 57: unconnected-(U6-PD10-Pad57) -> /LB
Routing:
- net /LB: track 0.00 -> 32.9 mm, vias 0 -> 2
- net /LG: track 0.00 -> 25.8 mm, vias 0 -> 2
- net /LR: track 0.00 -> 18.8 mm, vias 0 -> 2
- net /ISEN_60: track 15.3 -> 0.00 mm, vias 3 -> 0
- net PRI_LO: track 30.7 -> 46.0 mm, vias 2 -> 5
- net Net-(J8-Pin_2): track 0.00 -> 11.0 mm
- net Net-(J9-Pin_2): track 0.00 -> 10.8 mm
- net Net-(J10-Pin_2): track 0.00 -> 10.4 mm
- net Net-(J8-Pin_1): track 0.00 -> 7.78 mm
- net Net-(J10-Pin_1): track 0.00 -> 6.33 mm
- net Net-(J9-Pin_1): track 0.00 -> 6.31 mm
- net Net-(R75-Pad1): track 0.00 -> 3.49 mm
- net Net-(R79-Pad1): track 0.00 -> 2.30 mm
- net Net-(R77-Pad1): track 0.00 -> 2.30 mm
- net /AUX_I2S_WS: track 20.7 -> 20.0 mm

Commit message: file sync
Parts:
- removed C51, C52, C53, C54, C56: 100nF, Capacitor_SMD:C_0603_1608Metric
- removed C57: 10nF, Capacitor_SMD:C_0603_1608Metric
- removed C58: 10uF, Capacitor_SMD:C_0603_1608Metric
- removed C59: 1uF, Capacitor_SMD:C_0603_1608Metric
- added X2: 12.288MHz, Crystal:Crystal_SMD_2016-4Pin_2.0x1.6mm, F.Cu at (71.1, 65.0)
- D9: footprint Diode_SMD:D_1206_3216Metric -> Footprints:SOD-323HE
- moved J11 137.5 mm to (118.6, 81.3)
- moved R82 98.2 mm to (99.3, 72.4), turned to 180 degrees
- moved C83 98.0 mm to (96.5, 74.7), turned to 90 degrees
- moved C88 97.5 mm to (99.8, 74.9), turned to 90 degrees
- moved C50 97.1 mm to (80.8, 64.5)
- moved R86 96.5 mm to (99.3, 77.5)
- moved U16 96.0 mm to (104.1, 75.2), turned to 90 degrees
- moved R83 95.8 mm to (101.6, 74.2), turned to 90 degrees
- moved R81 95.7 mm to (97.8, 81.8), turned to 90 degrees
- moved C84 95.6 mm to (98.0, 74.7), turned to 90 degrees
- moved R85 95.1 mm to (101.6, 77.2), turned to -90 degrees
- moved C86 90.2 mm to (101.6, 71.1), turned to -90 degrees
- moved L10 88.3 mm to (114.3, 74.7), turned to -90 degrees
- moved R84 86.9 mm to (109.2, 71.4)
- moved C85 85.8 mm to (119.6, 74.6), turned to -90 degrees
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Connections:
- U6 pad 66: /HUM_SDA -> Net-(U6-PC9)
- U6 pad 67: /HUM_SCK -> unconnected-(U6-PA8-Pad67)
- U6 pad 93: unconnected-(U6-PB7-Pad93) -> /HUM_SDA
- U6 pad 95: unconnected-(U6-PB8-Pad95) -> /HUM_SCK
Routing:
- net +3V3: track 257.1 -> 454.3 mm, vias 9 -> 25
- net GND: track 194.1 -> 259.9 mm, vias 153 -> 258
- net +BATT: track 314.4 -> 366.6 mm, vias 17 -> 23
- net /HUM_SDA: track 1.81 -> 45.2 mm, vias 0 -> 2
- net /HUM_SCK: track 1.91 -> 42.8 mm, vias 0 -> 2
- net +15V: track 0.00 -> 25.7 mm, vias 0 -> 4
- net Net-(U6-NRST): track 0.00 -> 16.1 mm, vias 0 -> 2
- net PRI_LO: track 46.0 -> 30.7 mm, vias 5 -> 2
- net Net-(U6-PC9): track 0.00 -> 15.1 mm, vias 0 -> 2
- net /ISEN_60: track 0.00 -> 14.8 mm, vias 0 -> 3
- net /L+: track 4.46 -> 17.5 mm, vias 0 -> 2
- net Net-(D15-K): track 0.00 -> 12.0 mm
- net Net-(Q12-G): track 0.00 -> 11.3 mm
- net Net-(U16-COMP): track 0.00 -> 11.2 mm, vias 0 -> 2
- net Net-(Q12-S): track 0.00 -> 10.7 mm, vias 0 -> 2
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